File: hardware/kicad/gateway_esp32/gateway_esp32.kicad_sch (KiCad schematic)
At the start: 4 parts, among them J1 USB-C 5V power-only ou termin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, SW1 Botao reset EN (NA), U1 ESP32-DevKitC-32E

Commit message: Layouts finish, BM832A migration, fab package, quote, docs and status report
Parts:
- U1: footprint Connector_PinHeader_2.54mm:PinHeader_2x19_P2.54mm_Vertical -> nibas_gateway:ESP32-DevKitC-32E_Carrier
Changed lines of the file:
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@@
     (property "Reference" "U1" (at 177.8 124.46000000000001 0) (effects (font (size 1.27 1.27)) (justify left)))
     (property "Value" "ESP32-DevKitC-32E" (at 177.8 181.61 0) (effects (font (size 1.27 1.27)) (justify left)))
-    (property "Footprint" "Connector_PinHeader_2.54mm:PinHeader_2x19_P2.54mm_Vertical" (at 177.8 162.56 0) (effects (font (size 1.27 1.27)) (justify left)) (hide yes))
+    (property "Footprint" "nibas_gateway:ESP32-DevKitC-32E_Carrier" (at 177.8 162.56 0) (effects (font (size 1.27 1.27)) (justify left)) (hide yes))
     (property "Datasheet" "https://docs.espressif.com/projects/esp-dev-kits/en/latest/esp32/esp32-devkitc/user_guide.html" (at 177.8 165.1 0) (effects (font (size 1.27 1.27)) (justify left)) (hide yes))
     (pin "J2-1")
